Commit message: use a different color for each leg pair

File: data/LegAssembly.xacro (robot description, xacro)
@@ -6,5 +6,5 @@
  <xacro:property name="pi" value="3.1415926535897931" />
  <!-- Measurements and lables were taken from http://files.tested.com/photos/2015/04/05/74549-leg-measurement.jpg -->
-<xacro:macro name="strandbeest_leg" params="prefix">
+<xacro:macro name="strandbeest_leg" params="prefix material">
   <link name="${prefix}_bar_j">
     <inertial>
@@ -18,7 +18,5 @@
         <cylinder length="0.50" radius="0.01"/>
       </geometry>
-      <material name="orange">
-        <color rgba="1 .6392 .0980 1"/>
-      </material>
+      <material name="${material}"/>
     </visual>
   </link>
@@ -34,5 +32,5 @@
         <cylinder length="0.619" radius="0.01"/>
       </geometry>
-      <material name="orange"/>
+      <material name="${material}"/>
     </visual>
   </link>
@@ -55,5 +53,5 @@
         <cylinder length="0.393" radius="0.01"/>
       </geometry>
-      <material name="orange"/>
+      <material name="${material}"/>
     </visual>
   </link>
@@ -76,5 +74,5 @@
         <cylinder length="0.49" radius="0.01"/>
       </geometry>
-      <material name="orange"/>
+      <material name="${material}"/>
     </visual>
     <visual>
@@ -83,5 +81,5 @@
         <cylinder length="0.367" radius="0.01"/>
       </geometry>
-      <material name="orange"/>
+      <material name="${material}"/>
     </visual>
     <visual>
@@ -90,5 +88,5 @@
         <cylinder length="0.657" radius="0.01"/>
       </geometry>
-      <material name="orange"/>
+      <material name="${material}"/>
     </visual>
     <collision>
@@ -122,5 +120,5 @@
         <cylinder length="0.558" radius="0.01"/>
       </geometry>
-      <material name="orange"/>
+      <material name="${material}"/>
     </visual>
     <visual>
@@ -129,5 +127,5 @@
         <cylinder length="0.401" radius="0.01"/>
       </geometry>
-      <material name="orange"/>
+      <material name="${material}"/>
     </visual>
     <visual>
@@ -136,5 +134,5 @@
         <cylinder length="0.415" radius="0.01"/>
       </geometry>
-      <material name="orange"/>
+      <material name="${material}"/>
     </visual>
   </link>
@@ -162,5 +160,5 @@
         <cylinder length="0.394" radius="0.01"/>
       </geometry>
-      <material name="orange"/>
+      <material name="${material}"/>
     </visual>
   </link>

File: data/LegPair.xacro (robot description, xacro)
@@ -7,5 +7,5 @@
  <xacro:include filename="LegAssembly.xacro" />
  <xacro:property name="pi" value="3.1415926535897931" />
-  <xacro:macro name="strandbeest_leg_pair" params="prefix">
+  <xacro:macro name="strandbeest_leg_pair" params="prefix material">
   <link name="${prefix}_bar_l">
     <inertial>
@@ -19,5 +19,5 @@
         <cylinder length="0.078" radius="0.01"/>
       </geometry>
-      <material name="orange"/>
+      <material name="${material}"/>
     </visual>
   </link>
@@ -33,5 +33,5 @@
         <cylinder length="0.76" radius="0.01"/>
       </geometry>
-      <material name="orange"/>
+      <material name="${material}"/>
     </visual>
   </link>
@@ -53,8 +53,8 @@
         <cylinder length="0.15" radius="0.01"/>
       </geometry>
-      <material name="orange"/>
+      <material name="${material}"/>
     </visual>
   </link>
-  <xacro:strandbeest_leg prefix="${prefix}_leg1">
+  <xacro:strandbeest_leg prefix="${prefix}_leg1" material="${material}">
   </xacro:strandbeest_leg>
   <loop_joint name="${prefix}_leg1_loop_a_c" type="continuous">
@@ -69,5 +69,5 @@
     <origin rpy="0 0 0" xyz="0 0 0.15"/>
   </joint>
-  <xacro:strandbeest_leg prefix="${prefix}_leg2">
+  <xacro:strandbeest_leg prefix="${prefix}_leg2" material="${material}">
   </xacro:strandbeest_leg>
   <loop_joint name="${prefix}_leg2_loop_a_c" type="continuous">

File: data/Strandbeest.xacro (robot description, xacro)
@@ -6,4 +6,10 @@
  <xacro:include filename="LegPair.xacro" />
  <xacro:property name="pi" value="3.1415926535897931" />
+  <material name="#FF9619"> <color rgba="1.0 0.5882353 0.098039225 1"/> </material>
+  <material name="#FE6860"> <color rgba="0.9960785 0.40784317 0.37647063 1"/> </material>
+  <material name="#D2588C"> <color rgba="0.8235295 0.34509805 0.54901963 1"/> </material>
+  <material name="#8C5C99"> <color rgba="0.54901963 0.36078432 0.6 1"/> </material>
+  <material name="#4A5782"> <color rgba="0.2901961 0.34117648 0.50980395 1"/> </material>
+  <material name="#2F4858"> <color rgba="0.18431373 0.28235295 0.34509805 1"/> </material>
  <link name="crossbar">
     <inertial>
@@ -47,6 +53,6 @@
     <mechanicalReduction>1</mechanicalReduction>
   </transmission>
-  <xacro:macro name="positioned_leg_pair" params="name offset angle">
-	  <xacro:strandbeest_leg_pair prefix="${name}">
+  <xacro:macro name="positioned_leg_pair" params="name offset angle material">
+	  <xacro:strandbeest_leg_pair prefix="${name}" material="${material}">
 	  </xacro:strandbeest_leg_pair>
 	  <joint name="${name}_joint_crossbar_l" type="fixed">
@@ -68,15 +74,15 @@
   </loop_joint>
 	</xacro:macro>
-	<xacro:positioned_leg_pair name="pair01" offset="-0.5" angle="0">
+	<xacro:positioned_leg_pair name="pair01" offset="-0.5" angle="0" material="#2F4858">
 	</xacro:positioned_leg_pair>
-	<xacro:positioned_leg_pair name="pair02" offset="-0.3" angle="${2*pi/3}">
+	<xacro:positioned_leg_pair name="pair02" offset="-0.3" angle="${2*pi/3}" material="#4A5782">
 	</xacro:positioned_leg_pair>
-	<xacro:positioned_leg_pair name="pair03" offset="-0.1" angle="${4*pi/3}">
+	<xacro:positioned_leg_pair name="pair03" offset="-0.1" angle="${4*pi/3}" material="#8C5C99">
 	</xacro:positioned_leg_pair>
-	<xacro:positioned_leg_pair name="pair04" offset="0.1" angle="${pi/3}">
+	<xacro:positioned_leg_pair name="pair04" offset="0.1" angle="${pi/3}" material="#D2588C">
 	</xacro:positioned_leg_pair>
-	<xacro:positioned_leg_pair name="pair05" offset="0.3" angle="${3*pi/3}">
+	<xacro:positioned_leg_pair name="pair05" offset="0.3" angle="${3*pi/3}" material="#FE6860">
 	</xacro:positioned_leg_pair>
-	<xacro:positioned_leg_pair name="pair06" offset="0.5" angle="${5*pi/3}">
+	<xacro:positioned_leg_pair name="pair06" offset="0.5" angle="${5*pi/3}" material="#FF9619">
 	</xacro:positioned_leg_pair>
 </robot>
